Commit message: update apperance

File: urdf/rpo.urdf (robot description, URDF)
Before this commit: robot rpourdf, 24 links, 23 joints
Links:
- link base_link: mass 5.51295532 -> 4.5827
- link left_ankle_pitch_link: mass 0.084 -> 0.0366
- link left_ankle_roll_link: mass 0.33517651 -> 0.6208
- link left_arm_pitch_link: mass 0.47284363 -> 0.4686
- link left_arm_roll_link: mass 0.08401883 -> 0.1267
- link left_arm_yaw_link: mass 1.15324354 -> 1.1895
- link left_elbow_pitch_link: mass 0.09168684 -> 0.1113
- link left_elbow_yaw_link: mass 0.68145595 -> 0.7646
- link left_knee_link: mass 1.70223945 -> 2.0079
- link left_thigh_pitch_link: mass 2.34600715 -> 2.5516
- link left_thigh_roll_link: mass 1.66236465 -> 1.8661
- link left_thigh_yaw_link: mass 1.71784575 -> 1.8739
- link right_ankle_pitch_link: mass 0.084 -> 0.0366
- link right_ankle_roll_link: mass 0.33517651 -> 0.6208
- link right_arm_pitch_link: mass 0.47284363 -> 0.4686
- link right_arm_roll_link: mass 0.08401883 -> 0.1080
- link right_arm_yaw_link: mass 1.15429959 -> 1.1895
- link right_elbow_pitch_link: mass 0.09168684 -> 0.1113
- link right_elbow_yaw_link: mass 0.68145595 -> 0.6296
- link right_knee_link: mass 1.70223945 -> 1.9878
- link right_thigh_pitch_link: mass 2.34600715 -> 2.5517
- link right_thigh_roll_link: mass 1.66310652 -> 1.8665
- link right_thigh_yaw_link: mass 1.71632614 -> 1.8739
- link torso_link: mass 7.58189737 -> 9.6686
Joints:
- joint left_ankle_pitch_joint: origin xyz=0 -0.02085 -0.3 rpy=0 0 0 -> xyz=0 -0.01885 -0.3 rpy=0 0 0
- joint left_arm_pitch_joint: origin xyz=0 0.121749999999383 0.206175860782433 rpy=0 0 0 -> xyz=0 0.12175 0.20818 rpy=0 0 0
- joint left_arm_roll_joint: origin xyz=0.0200000000000018 0.056 0 rpy=0 0 0 -> xyz=0.02 0.056 0 rpy=0 0 0
- joint left_arm_yaw_joint: origin xyz=-0.0200000000000002 0 -0.049999999999998 rpy=0 0 0 -> xyz=-0.02 0 -0.05 rpy=0 0 0
- joint left_elbow_pitch_joint: origin xyz=0 0.0199999999999982 -0.188749999999997 rpy=0 0 0 -> xyz=0 0.02 -0.18875 rpy=0 0 0
- joint left_elbow_yaw_joint: origin xyz=0.0499999999999968 -0.0199999999999994 0 rpy=0 0 0 -> xyz=0.04975 -0.02 0 rpy=0 0 0
- joint left_thigh_pitch_joint: origin xyz=0.060622 0.02085 -0.035 rpy=0 0 0 -> xyz=0.062354 0.01885 -0.036 rpy=0 -5.3117E-05 0
- joint left_thigh_roll_joint: origin xyz=-0.017693 0 -0.072346 rpy=0 0 0 -> xyz=-0.019425 0 -0.071346 rpy=0 0 0
- joint left_thigh_yaw_joint: origin xyz=-0.071093 0.0725 -0.051778 rpy=0 0 0 -> xyz=-0.031149 0.0725 0.017407 rpy=0 0 0
- joint right_ankle_pitch_joint: origin xyz=0 0.0208500000000073 -0.299999999999986 rpy=0 0 0 -> xyz=0 0.01885 -0.3 rpy=0 0 0
- joint right_ankle_roll_joint: axis 1 0 0 -> 1 0 5.3117E-05; origin xyz=0 0 0 rpy=0 0 0 -> xyz=0 0 0 rpy=0 -5.3117E-05 0
- joint right_arm_pitch_joint: origin xyz=0 -0.121750000000346 0.206175860781721 rpy=0 0 0 -> xyz=0 -0.12175 0.20818 rpy=0 0 0
- joint right_arm_roll_joint: origin xyz=0.0200000000000407 -0.056 0 rpy=0 0 0 -> xyz=0.02 -0.056 0 rpy=0 0 0
- joint right_arm_yaw_joint: origin xyz=-0.02 0 -0.0500000000000019 rpy=0 0 0 -> xyz=-0.02 0 -0.05 rpy=0 0 0
- joint right_elbow_pitch_joint: origin xyz=0 -0.0200000000000019 -0.18875 rpy=0 0 0 -> xyz=0 -0.02 -0.18875 rpy=0 0 0
- joint right_elbow_yaw_joint: origin xyz=0.0500000000000002 0.0200000000000004 0 rpy=0 0 0 -> xyz=0.05 0.02 0 rpy=0 0 0
- joint right_knee_joint: origin xyz=0 0 -0.250000000000016 rpy=0 0 0 -> xyz=-0.0030239 0 -0.24998 rpy=0 0.012096 0
- joint right_thigh_pitch_joint: origin xyz=0.0619208163652291 -0.0208499999999942 -0.0357500000093095 rpy=0 0 0 -> xyz=0.062354 -0.01885 -0.036 rpy=0 -0.012096 0
- joint right_thigh_roll_joint: origin xyz=-0.0189924084475403 0 -0.0715958163677252 rpy=0 0 0 -> xyz=-0.019675 0 -0.071779 rpy=0 0 0
- joint right_thigh_yaw_joint: origin xyz=-0.071093 -0.0725 -0.051778 rpy=0 0 0 -> xyz=-0.030899 -0.0725 0.01784 rpy=0 0 0
- joint torso_joint: origin xyz=-0.0281649492242451 0 0.0672000000054882 rpy=0 0 0 -> xyz=0.011779 0 0.13439 rpy=0 0 0
